File: D3_Face/D3_Face.kicad_pcb (KiCad board)
At the start: 2 copper layers, 100 x 70 mm, 31 parts, among them J1 Conn_01x05_Male, U1 MAX7219, U2 MAX7219, U3 MAX7219, U4 MAX7219, U5 MAX7219, U6 MAX7219

Commit message: finish Face PCB traces
Parts:
- moved U4 132.3 mm to (114.0, 88.5), turned to 90 degrees
- moved C10 91.1 mm to (116.0, 73.0), turned to 180 degrees
- moved U5 89.8 mm to (146.1, 88.5), turned to 90 degrees
- moved C7 80.7 mm to (108.9, 75.4), turned to 180 degrees
- moved R4 79.7 mm to (88.5, 75.6)
- moved C12 77.0 mm to (148.0, 73.0), turned to 180 degrees
- moved C11 76.9 mm to (179.0, 72.8), turned to 180 degrees
- moved R5 71.1 mm to (120.8, 75.4)
- moved R6 69.8 mm to (152.7, 75.4)
- moved C8 53.0 mm to (140.8, 75.4), turned to 180 degrees
- moved C9 52.6 mm to (173.0, 75.4), turned to 180 degrees
- moved U6 49.5 mm to (178.1, 88.4), turned to 90 degrees
Routing:
- net CS: track 53.2 -> 189.0 mm
- net Net-(U3-Pad24): track 0.00 -> 121.4 mm, vias 0 -> 1
- net CLK: track 96.5 -> 178.4 mm
- net Net-(U5-Pad24): track 0.00 -> 38.2 mm, vias 0 -> 1
- net Net-(U4-Pad24): track 0.00 -> 37.9 mm, vias 0 -> 1
- net Net-(D5-Pad5): track 0.00 -> 36.7 mm
- net Net-(D4-Pad5): track 0.00 -> 36.1 mm
- net Net-(D6-Pad5): track 0.00 -> 36.0 mm
- net Net-(D5-Pad11): track 0.00 -> 35.0 mm
- net Net-(D6-Pad11): track 0.00 -> 35.0 mm
- net Net-(D4-Pad11): track 0.00 -> 34.5 mm
- net Net-(D4-Pad9): track 0.00 -> 30.1 mm
- net Net-(D5-Pad9): track 0.00 -> 30.1 mm
- net Net-(D6-Pad9): track 0.00 -> 29.6 mm
- net Net-(D4-Pad6): track 0.00 -> 24.9 mm
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
Commit message: Create D3_Board
Parts:
- removed D1, D2, D3, D4, D5, D6: Matrix_LED_8x8, D3_Face:Matrix_LED_8x8
- added LED1: Matrix_LED_8x8, D3_Face:Matrix_LED_8x8, F.Cu at (120.0, 80.0)
- added LED2: Matrix_LED_8x8, D3_Face:Matrix_LED_8x8, F.Cu at (152.0, 80.0)
- added LED3: Matrix_LED_8x8, D3_Face:Matrix_LED_8x8, F.Cu at (184.0, 80.0)
- added LED4: Matrix_LED_8x8, D3_Face:Matrix_LED_8x8, F.Cu at (120.0, 112.0)
- added LED5: Matrix_LED_8x8, D3_Face:Matrix_LED_8x8, F.Cu at (152.0, 112.0)
- added LED6: Matrix_LED_8x8, D3_Face:Matrix_LED_8x8, F.Cu at (184.0, 112.0)
- moved C12 57.0 mm to (195.8, 104.0), turned to 0 degrees
- moved J1 36.1 mm to (105.9, 90.9)
- moved C6 35.6 mm to (195.8, 72.0), turned to 0 degrees
- moved R2 35.3 mm to (140.6, 72.0)
- moved R3 35.3 mm to (172.6, 72.0)
- moved C4 35.2 mm to (131.8, 72.0), turned to 0 degrees
- moved C5 35.1 mm to (163.8, 72.0), turned to 0 degrees
- moved U6 34.8 mm to (198.0, 117.0)
- moved U5 34.8 mm to (166.0, 117.0)
- moved U1 34.8 mm to (134.0, 85.0)
- moved U2 34.8 mm to (166.0, 85.0)
- moved U4 34.8 mm to (134.0, 117.0)
- moved R4 34.8 mm to (108.6, 104.0)
- moved R6 34.8 mm to (172.6, 104.0)
- moved C10 34.8 mm to (131.8, 104.0), turned to 0 degrees
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Routing:
- net CLK: track 178.4 -> 222.5 mm, vias 1 -> 0
- net CS: track 189.0 -> 217.2 mm
- net Net-(LED3-Pad8): track 35.4 -> 11.5 mm
- net Net-(LED5-Pad8): track 35.0 -> 11.5 mm
- net Net-(LED6-Pad8): track 35.0 -> 11.5 mm
- net Net-(LED4-Pad8): track 34.5 -> 11.5 mm
- net Net-(LED1-Pad8): track 34.0 -> 11.5 mm
- net Net-(LED2-Pad8): track 33.9 -> 11.5 mm
- net Net-(LED3-Pad11): track 38.0 -> 17.5 mm
- net Net-(LED5-Pad11): track 36.7 -> 17.5 mm
- net Net-(LED1-Pad11): track 36.7 -> 17.5 mm
- net Net-(LED2-Pad11): track 36.5 -> 17.5 mm
- net Net-(LED4-Pad11): track 36.1 -> 17.5 mm
- net Net-(LED6-Pad11): track 36.0 -> 17.5 mm
- net Net-(LED1-Pad15): track 25.5 -> 10.4 mm
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Other:
- board outline removed

Commit message: Finish PCBs
Parts:
- added G***: LOGO, D3_Board:ieee_logo_11_8mm, B.Cu at (136.0, 94.4)
- added G***: LOGO, D3_Board:ras_logo_11_8mm, B.Cu at (168.0, 94.1)
- added G***: LOGO, D3_Board:ras_logo_11_8mm, F.Cu at (168.0, 93.5)
- added G***: LOGO, D3_Board:ieee_logo_11_8mm, F.Cu at (136.0, 93.6)
- added REF**: MountingHole_4.5mm_Pad, MountingHole:MountingHole_4.5mm_Pad, F.Cu at (106.5, 65.5)
- added REF**: MountingHole_4.5mm_Pad, MountingHole:MountingHole_4.5mm_Pad, F.Cu at (197.5, 65.5)
- added REF**: MountingHole_4.5mm_Pad, MountingHole:MountingHole_4.5mm_Pad, F.Cu at (197.5, 126.5)
- added REF**: MountingHole_4.5mm_Pad, MountingHole:MountingHole_4.5mm_Pad, F.Cu at (106.5, 126.5)
Routing:
- net Net-(U3-Pad24): track 121.5 -> 118.9 mm
- net CS: track 217.2 -> 216.4 mm
- net CLK: track 222.5 -> 221.8 mm
Other:
- board outline added: 100 x 70 mm
