File: D3_Board/_autosave-D3_Board.kicad_pcb (KiCad board)
At the start: 2 copper layers, 115 x 83 mm, 42 parts, among them J1 POWER_IN, J10 ACS_SENSOR, J11 H-BRIDGE1, J12 H-BRIDGE2, J13 BUZZER, J14 MOTOR1_POW, J15 MOTOR1_OUT, J16 MOTOR2_POW, J17 MOTOR2_OUT, J2 POWER_IN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

Commit message: Finish traces
Routing:
- net +5V: track 43.9 -> 47.0 mm
Other:
- board text added: "I3E-D3 Board"
Changed lines of the file:
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@@
   (general
     (thickness 1.6)
-    (drawings 4)
-    (tracks 347)
+    (drawings 5)
+    (tracks 349)
     (zones 0)
     (modules 42)
@@
   (layers
     (0 F.Cu signal hide)
-    (31 B.Cu signal hide)
+    (31 B.Cu signal)
     (32 B.Adhes user)
     (33 F.Adhes user)
@@
     )
   )
+  (gr_text "I3E-D3 Board" (at 13.9065 16.51) (layer F.SilkS)
+    (effects (font (size 2 2) (thickness 0.5)))
+  )
   (gr_line (start 115 0) (end 115 83) (layer Edge.Cuts) (width 0.1))
   (gr_line (start 0 0) (end 115 0) (layer Edge.Cuts) (width 0.1))
@@
   (segment (start 75.057 45.085) (end 73.025 47.117) (width 0.25) (layer B.Cu) (net 3))
   (segment (start 75.057 41.529) (end 75.057 45.085) (width 0.25) (layer B.Cu) (net 3))
-  (segment (start 72.5932 35.0012) (end 72.5932 33.5915) (width 0.25) (layer F.Cu) (net 3))
+  (segment (start 87.249 19.177) (end 85.7885 19.177) (width 0.25) (layer F.Cu) (net 3))
+  (segment (start 87.249 19.177) (end 85.6615 19.177) (width 0.25) (layer F.Cu) (net 3))
   (segment (start 72.94497 35.35297) (end 72.5932 35.0012) (width 0.25) (layer F.Cu) (net 3))
   (segment (start 79.13753 35.35297) (end 72.94497 35.35297) (width 0.25) (layer F.Cu) (net 3))
-  (segment (start 80.529019 33.961481) (end 79.13753 35.35297) (width 0.25) (layer F.Cu) (net 3))
-  (segment (start 80.529019 24.436481) (end 80.529019 33.961481) (width 0.25) (layer F.Cu) (net 3))
-  (segment (start 85.7885 19.177) (end 80.529019 24.436481) (width 0.25) (layer F.Cu) (net 3))
-  (segment (start 87.249 19.177) (end 85.7885 19.177) (width 0.25) (layer F.Cu) (net 3))
+  (segment (start 80.8355 33.655) (end 79.13753 35.35297) (width 0.25) (layer F.Cu) (net 3))
+  (segment (start 80.8355 24.0665) (end 80.8355 33.655) (width 0.25) (layer F.Cu) (net 3))
+  (segment (start 85.725 19.177) (end 80.8355 24.0665) (width 0.25) (layer F.Cu) (net 3))
+  (segment (start 72.5932 35.0012) (end 72.5932 33.5915) (width 0.25) (layer F.Cu) (net 3))
+  (segment (start 87.249 19.177) (end 85.725 19.177) (width 0.25) (layer F.Cu) (net 3))
   (segment (start 85.09 41.3385) (end 87.9475 41.3385) (width 0.25) (layer B.Cu) (net 4))
   (segment (start 103.251 56.642) (end 105.029 56.642) (width 0.25) (layer B.Cu) (net 4))
@@
   (segment (start 94.7966 7.239) (end 94.7966 9.3434) (width 0.25) (layer B.Cu) (net 20))
   (segment (start 44.35475 12.03325) (end 42.1132 14.2748) (width 0.25) (layer B.Cu) (net 20))
+  (segment (start 99.7966 7.0485) (end 99.7966 6.0735) (width 2.286) (layer B.Cu) (net 21))
   (segment (start 99.7966 6.0735) (end 95.6281 1.905) (width 2.286) (layer B.Cu) (net 21))
-  (segment (start 99.7966 7.0485) (end 99.7966 6.0735) (width 2.286) (layer B.Cu) (net 21))
+  (segment (start 42.799 1.905) (end 41.101 3.603) (width 2.286) (layer B.Cu) (net 21))
+  (segment (start 41.101 3.603) (end 41.101 5.9) (width 2.286) (layer B.Cu) (net 21))
   (segment (start 95.6281 1.905) (end 42.799 1.905) (width 2.286) (layer B.Cu) (net 21))
-  (segment (start 41.101 3.603) (end 41.101 5.9) (width 2.286) (layer B.Cu) (net 21))
-  (segment (start 42.799 1.905) (end 41.101 3.603) (width 2.286) (layer B.Cu) (net 21))
   (segment (start 34.6075 33.7058) (end 34.4932 33.5915) (width 0.25) (layer F.Cu) (net 22))
   (segment (start 102.489 20.5105) (end 102.489 19.177) (width 0.25) (layer F.Cu) (net 22))
