File: D3_Board/D3_Board.kicad_pcb (KiCad board)
At the start: 2 copper layers, 1 part, among them U1 YAAJ_DCDC_StepUp_SX1308

Commit message: PCB Layout inprog
Parts:
- added C1: 1000uF, Capacitor_THT:CP_Radial_D10.0mm_P5.00mm, F.Cu at (12.4, 39.8)
- added J1: POWER_IN, Connector_AMASS:AMASS_XT60-M_1x02_P7.20mm_Vertical, F.Cu at (28.8, 77.3)
- added J10: ACS_SENSOR, Connector_PinHeader_2.54mm:PinHeader_1x03_P2.54mm_Vertical, F.Cu at (9.65, 22.4)
- added J11: H-BRIDGE1, Connector_PinHeader_2.54mm:PinHeader_1x07_P2.54mm_Vertical, F.Cu at (87.2, 19.2)
- added J12: H-BRIDGE2, Connector_PinHeader_2.54mm:PinHeader_1x07_P2.54mm_Vertical, F.Cu at (87.2, 14.4)
- added J13: BUZZER_PIN, Connector_PinHeader_2.54mm:PinHeader_1x02_P2.54mm_Vertical, F.Cu at (105.2, 70.2)
- added J14: MOTOR1_POWER, TerminalBlock_Phoenix:TerminalBlock_Phoenix_PT-1,5-2-5.0-H_1x02_P5.00mm_Horizontal, F.Cu at (32.9, 5.90)
- added J15: MOTOR1_OUT, TerminalBlock_Phoenix:TerminalBlock_Phoenix_PT-1,5-2-5.0-H_1x02_P5.00mm_Horizontal, F.Cu at (56.2, 5.90)
- added J16: MOTOR2_POW, TerminalBlock_Phoenix:TerminalBlock_Phoenix_PT-1,5-2-5.0-H_1x02_P5.00mm_Horizontal, F.Cu at (22.8, 5.90)
- added J17: MOTOR2_OUT, TerminalBlock_Phoenix:TerminalBlock_Phoenix_PT-1,5-2-5.0-H_1x02_P5.00mm_Horizontal, F.Cu at (46.1, 5.90)
- added J2: POWER_IN, TerminalBlock_Phoenix:TerminalBlock_Phoenix_PT-1,5-2-5.0-H_1x02_P5.00mm_Horizontal, F.Cu at (44.6, 76.8)
- added J3: RASPBERRY_POWER_IN, TerminalBlock_Phoenix:TerminalBlock_Phoenix_PT-1,5-2-5.0-H_1x02_P5.00mm_Horizontal, F.Cu at (60.2, 76.8)
- added J4: Raspberry_connection, Connector_PinHeader_2.54mm:PinHeader_1x04_P2.54mm_Vertical, F.Cu at (105.0, 56.6)
- added J5: CURRENT_POWER_IN, TerminalBlock_Phoenix:TerminalBlock_Phoenix_PT-1,5-2-5.0-H_1x02_P5.00mm_Horizontal, F.Cu at (15.4, 77.2)
- added J6: LED_Matrix, Connector_PinHeader_2.54mm:PinHeader_1x05_P2.54mm_Vertical, F.Cu at (99.9, 26.7)
- added J7: USB_TTL, Connector_PinHeader_2.54mm:PinHeader_1x06_P2.54mm_Vertical, F.Cu at (89.9, 79.8)
- added J8: MOTOR1, Connector_JST:JST_EH_B6B-EH-A_1x06_P2.50mm_Vertical, F.Cu at (81.3, 6.54)
- added J9: MOTOR2, Connector_JST:JST_EH_B6B-EH-A_1x06_P2.50mm_Vertical, F.Cu at (99.8, 6.54)
- added M1: Motor_Servo, Connector_PinHeader_2.54mm:PinHeader_1x03_P2.54mm_Vertical, F.Cu at (78.7, 66.2)
- added M2: Motor_Servo, Connector_PinHeader_2.54mm:PinHeader_1x03_P2.54mm_Vertical, F.Cu at (78.5, 49.4)
- added Q1: BC546, Package_TO_SOT_THT:TO-92_Inline, F.Cu at (56.6, 60.8)
- added Q2: BC546, Package_TO_SOT_THT:TO-92_Inline, F.Cu at (56.6, 44.1)
- added Q3: BC546, Package_TO_SOT_THT:TO-92_Inline, F.Cu at (56.6, 67.2)
- added Q4: BC546, Package_TO_SOT_THT:TO-92_Inline, F.Cu at (56.6, 50.4)
- added R1: 11k, Resistor_THT:R_Axial_DIN0207_L6.3mm_D2.5mm_P10.16mm_Horizontal, F.Cu at (23.1, 44.0)
- added R10: 3.3k, Resistor_THT:R_Axial_DIN0207_L6.3mm_D2.5mm_P10.16mm_Horizontal, F.Cu at (21.8, 35.1)
- added R2: 3.3k, Resistor_THT:R_Axial_DIN0207_L6.3mm_D2.5mm_P10.16mm_Horizontal, F.Cu at (33.3, 39.9)
- added R3: 4.7k, Resistor_THT:R_Axial_DIN0207_L6.3mm_D2.5mm_P10.16mm_Horizontal, F.Cu at (62.9, 59.6)
- added R4: 4.7k, Resistor_THT:R_Axial_DIN0207_L6.3mm_D2.5mm_P10.16mm_Horizontal, F.Cu at (62.9, 43.1)
- added R5: 4.7k, Resistor_THT:R_Axial_DIN0207_L6.3mm_D2.5mm_P10.16mm_Horizontal, F.Cu at (62.9, 63.6)
- added R6: 4.7k, Resistor_THT:R_Axial_DIN0207_L6.3mm_D2.5mm_P10.16mm_Horizontal, F.Cu at (62.9, 47.1)
- added R7: 1k, Resistor_THT:R_Axial_DIN0207_L6.3mm_D2.5mm_P10.16mm_Horizontal, F.Cu at (73.0, 67.7)
- added R8: 1k, Resistor_THT:R_Axial_DIN0207_L6.3mm_D2.5mm_P10.16mm_Horizontal, F.Cu at (62.9, 51.2)
- added R9: 1.7k, Resistor_THT:R_Axial_DIN0207_L6.3mm_D2.5mm_P10.16mm_Horizontal, F.Cu at (17.7, 25.0)
- added REF**: MountingHole_4.5mm_Pad, MountingHole:MountingHole_4.5mm_Pad, F.Cu at (109.9, 5.08)
- added REF**: MountingHole_4.5mm_Pad, MountingHole:MountingHole_4.5mm_Pad, F.Cu at (109.9, 77.9)
- added REF**: MountingHole_4.5mm_Pad, MountingHole:MountingHole_4.5mm_Pad, F.Cu at (5.08, 77.9)
- added REF**: MountingHole_4.5mm_Pad, MountingHole:MountingHole_4.5mm_Pad, F.Cu at (5.08, 5.08)
- added U2: LM2596_module, D3_Board:LM2596_module, F.Cu at (27.2, 59.3)
- added U3: GPS_NEO6M_module, D3_Board:GPS_NEO6M_module, F.Cu at (98.6, 42.6)
- added U4: MPU6050_module, D3_Board:MPU6050_module, F.Cu at (92.1, 65.5)
- U1: value YAAJ_DCDC_StepUp_SX1308 -> ChinaBluePill-bluepill-D3_Board; footprint lm2596_module:lm2596_module -> BLUEPILL:BluePill_STM32F103C
- moved U1 221.3 mm to (29.5, 33.6), turned to 90 degrees
Connections:
- U1 pad 3: Net-(U1-Pad3) -> /MOTOR1_PWM
- U1 pad 4: Net-(U1-Pad4) -> /MOTOR2_PWM
Routing:
- net /TX_GPS: track 0.00 -> 26.3 mm
- net /RX_GPS: track 0.00 -> 26.3 mm
- net Net-(M1-Pad1): track 0.00 -> 25.6 mm
- net /SDA: track 0.00 -> 20.0 mm
- net /SCL: track 0.00 -> 20.0 mm
- net Net-(Q1-Pad1): track 0.00 -> 12.4 mm
- net Net-(J10-Pad2): track 0.00 -> 8.06 mm
- net Net-(Q1-Pad2): track 0.00 -> 7.03 mm
- net /ACS: track 0.00 -> 4.13 mm
- net /AVS: track 0.00 -> 4.06 mm
- added copper zone on F.Cu, net +5V
- added copper zone on B.Cu, net GND
Other:
- board outline added: 115 x 83 mm

Commit message: Finish traces
Parts:
- J13: value BUZZER_PIN -> BUZZER
- J14: value MOTOR1_POWER -> MOTOR1_POW
- J4: value Raspberry_connection -> RASPBERRY
- M1: value Motor_Servo -> SERVO2
- M2: value Motor_Servo -> SERVO1
- U1: value ChinaBluePill-bluepill-D3_Board -> Bluepill
- U2: value LM2596_module -> LM2596
- U3: value GPS_NEO6M_module -> GPS_NEO6M
- U4: value MPU6050_module -> MPU6050
- moved C1 2.18 mm to (14.2, 41.0)
- moved J9 1.21 mm to (99.9, 7.75)
- moved J8 1.14 mm to (81.3, 7.68)
Connections:
- U1 pad 35: /ENCODER2_A -> /ENCODER2_B
- U1 pad 36: /ENCODER2_B -> /ENCODER2_A
Routing:
- net /BUZZER: track 0.00 -> 173.4 mm
- net /CS_LED: track 0.00 -> 126.4 mm
- net /DOUT_LED: track 0.00 -> 120.9 mm
- net /CLK_LED: track 0.00 -> 119.1 mm
- net +12V: track 0.00 -> 104.9 mm
- net +3V3: track 0.00 -> 103.5 mm
- net /MOTOR2_PWM: track 0.00 -> 95.4 mm
- net /MOTOR1_PWM: track 0.00 -> 83.6 mm
- net /RX_SERIAL: track 0.00 -> 73.1 mm
- net /TX_SERIAL: track 0.00 -> 72.5 mm
- net Net-(C1-Pad1): track 0.00 -> 72.2 mm
- net /MOTOR2_M2: track 0.00 -> 64.4 mm
- net /ENCODER2_B: track 0.00 -> 60.9 mm
- net /MOTOR1_CS: track 0.00 -> 60.4 mm
- net /ENCODER2_A: track 0.00 -> 59.7 mm
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
Commit message: Finish PCBs
Parts:
- added G***: LOGO, D3_Board:ieee_logo_11_8mm, B.Cu at (106.7, 35.8)
- added G***: LOGO, D3_Board:ieee_logo, F.Cu at (99.1, 42.5)
- added G***: LOGO, D3_Board:ras_logo_11_8mm, B.Cu at (97.5, 35.6)
- added G***: LOGO, D3_Board:ras_logo, F.Cu at (34.3, 26.0)
- moved R2 1.27 mm to (33.2, 41.2)
- moved R1 1.21 mm to (23.1, 45.2)
Routing:
- net /AVS: track 63.2 -> 64.5 mm
- net Net-(C1-Pad1): track 72.2 -> 71.4 mm
Other:
- board text added: "12V"
- board text added: "5V"
- board text added: "BUZ"
- board text added: "CLK"
- board text added: "CS"
- board text added: "DO"
- board text added: "Developed by RAS CIMATEC Student Chapter"
- board text added: "EN"
- board text added: "GND"
- board text added: "I3E-D3 Board"
- board text added: "IN"
- board text added: "INA"
- board text added: "INB"
- board text added: "M1"
- board text added: "M2"
- board text added: "PWM"
- board text added: "RX"
- board text added: "RX_GPS"
- board text added: "SCL_IMU"
- board text added: "SDA_IMU"
- board text added: "SIG"
- board text added: "TX"
- board text added: "TX_GPS"
