File: D3_Board/D3_Board.sch (KiCad schematic (older format))
At the start: 2 parts, among them U1 BP

Commit message: Create D3_Board
Parts:
- removed C?: C, symbol Device:C
- removed U1: BP, BP:BLUEPILL, symbol bluepill:BP
- added J?: LED_Matrix, symbol Connector_Generic:Conn_01x05
- added J?: MOTOR1, symbol Connector_Generic:Conn_01x06
- added J?: MOTOR2, symbol Connector_Generic:Conn_01x06
- added M? (x2): Motor_Servo, Connector_PinHeader_2.54mm:PinHeader_1x03_P2.54mm_Vertical, symbol Motor:Motor_Servo
- added U?: ChinaBluePill, bluepill:BluePill_STM32F103C, symbol bluepill:ChinaBluePill
- added U? (x2): LM2596_module, symbol lm2596_module:YAAJ_DCDC_StepUp_SX1308
Connections:
- net labels added: +12V, +3.3V, CLK_LED, CS_LED, DOUT_LED, ENCODER1_A, ENCODER1_B, ENCODER2_A, ENCODER2_B, MOTOR1_M1, MOTOR1_M2, MOTOR2_M1, MOTOR2_M2, SERVO1, SERVO2
- wire segments 2 -> 41

Commit message: Board inprog
Parts:
- added J?: MOTOR1_POWER, TerminalBlock:TerminalBlock_Altech_AK300-2_P5.00mm, symbol Connector_Generic:Conn_01x02
- added J?: MOTOR1_OUT, TerminalBlock:TerminalBlock_Altech_AK300-2_P5.00mm, symbol Connector_Generic:Conn_01x02
- added J?: MOTOR2_POW, TerminalBlock:TerminalBlock_Altech_AK300-2_P5.00mm, symbol Connector_Generic:Conn_01x02
- added J?: MOTOR2_OUT, TerminalBlock:TerminalBlock_Altech_AK300-2_P5.00mm, symbol Connector_Generic:Conn_01x02
- added J?: MPU6050, Connector_PinHeader_2.54mm:PinHeader_1x08_P2.54mm_Vertical, symbol Connector_Generic:Conn_01x08
- added J?: POWER_IN, TerminalBlock:TerminalBlock_Altech_AK300-2_P5.00mm, symbol Connector_Generic:Conn_01x02
- added J?: H-BRIDGE1, Connector_PinHeader_2.54mm:PinHeader_1x07_P2.54mm_Vertical, symbol Connector_Generic:Conn_01x07
- added J?: H-BRIDGE2, Connector_PinHeader_2.54mm:PinHeader_1x07_P2.54mm_Vertical, symbol Connector_Generic:Conn_01x07
- added J?: RASPBERRY_POWER_IN, TerminalBlock:TerminalBlock_Altech_AK300-2_P5.00mm, symbol Connector_Generic:Conn_01x02
- added J?: Raspberry_Pi_2_3, Connector_PinHeader_2.54mm:PinHeader_2x20_P2.54mm_Vertical, symbol Connector:Raspberry_Pi_2_3
- added J?: ACS_SENSOR, Connector_PinHeader_2.54mm:PinHeader_1x03_P2.54mm_Vertical, symbol Connector_Generic:Conn_01x03
- added J?: GPS, Connector_PinHeader_2.54mm:PinHeader_1x04_P2.54mm_Vertical, symbol Connector_Generic:Conn_01x04
- added J?: BLUETOOTH, Connector_PinHeader_2.54mm:PinHeader_1x04_P2.54mm_Vertical, symbol Connector_Generic:Conn_01x04
- added R?: 1.7K, symbol Device:R
- added R?: 3.3K, symbol Device:R
- J2, J3: renamed from J?; footprint (none) -> Connector_PinHeader_2.54mm:PinHeader_1x06_P2.54mm_Vertical
- U1, U3: renamed from U?; footprint (none) -> LM2596:lm2596_module; symbol lm2596_module:YAAJ_DCDC_StepUp_SX1308 -> D3_Board:YAAJ_DCDC_StepUp_SX1308-lm2596_module
- U2: renamed from U?; footprint bluepill:BluePill_STM32F103C -> BLUEPILL:BluePill_STM32F103C; symbol bluepill:ChinaBluePill -> D3_Board:ChinaBluePill-bluepill
- gave numbers to parts that had none: 3
Connections:
- net labels added: ACS, MOTOR1_CS, MOTOR1_EN, MOTOR1_INA, MOTOR1_INB, MOTOR1_PWM, MOTOR2_CS, MOTOR2_EN, MOTOR2_INA, MOTOR2_INB, MOTOR2_PWM, SCL, SDA
- wire segments 41 -> 99
- no-connect marks 0 -> 4

Commit message: Add connections
Parts:
- added C?: CP, symbol Device:CP
- added J?: USB_TTL, Connector_PinHeader_2.54mm:PinHeader_1x06_P2.54mm_Vertical, symbol Connector_Generic:Conn_01x06
- J?: footprint Connector_PinHeader_2.54mm:PinHeader_1x04_P2.54mm_Vertical -> Connector_PinHeader_2.54mm:PinHeader_1x06_P2.54mm_Vertical; symbol Connector_Generic:Conn_01x04 -> Connector_Generic:Conn_01x06
Connections:
- net +12V: now also C?.1
- net +5V: now also J?.1 (Pin_1), J?.2 (Pin_2), U2.5V, J?.1 (Pin_1)
- net ACS: now also U2.PA8
- net CLK_LED: now also U2.PA5
- net CS_LED: now also U2.PA4
- net DOUT_LED: now also U2.PA7
- net ENCODER1_A: now also U2.PB12
- net ENCODER1_B: now also U2.PB13
- net ENCODER2_A: now also U2.PB14
- net ENCODER2_B: now also U2.PB15
- net GND: now also J?.3 (Pin_3), J?.4 (Pin_4), U2.GND, C?.2, J?.6 (Pin_6)
- net MOTOR1_CS: now also U2.PA0
- net MOTOR1_EN: now also U2.PA11, U2.PB3
- net MOTOR1_INA: now also U2.PA12, U2.PB4
- net MOTOR1_INB: now also U2.PA15, U2.PB5
- net MOTOR1_PWM: now also U2.PB8
- net MOTOR2_CS: now also U2.PA1
- net MOTOR2_PWM: now also U2.PB9
- net SCL: now also J?.5 (SCL/GPIO3)
- net SDA: now also J?.3 (SDA/GPIO2)
- net SERVO1: now also U2.PB6
- net SERVO2: now also U2.PB7
- net TX_SERIAL: now reaches U2.PA10
- net TX_SERIAL: now also J?.4 (Pin_4)
- net RX_BLUETOOTH: now reaches U2.PA2
- net RX_BLUETOOTH: now also J?.5 (Pin_5)
- net TX_BLUETOOTH: now reaches U2.PA3
- net TX_BLUETOOTH: now also J?.4 (Pin_4)
- net RX_SERIAL: now reaches U2.PA9
- net RX_SERIAL: now also J?.5 (Pin_5)
- net TX_GPS: now reaches J?.10 (GPIO15/RXD)
- net TX_GPS: now also J?.3 (Pin_3)
- net RX_GPS: now reaches J?.8 (GPIO14/TXD)
- net RX_GPS: now also J?.2 (Pin_2)
- no-connect marks 4 -> 8
Other:
- note added: "Alimentar o Raspberry \npela entrada USB\n"
- moved on the sheet: J1, J2, J3, J?, M1, M2, R?, U1, U2, U3

Commit message: Finish schematics
Parts:
- removed U3: LM2596_module, LM2596:lm2596_module, symbol D3_Board:YAAJ_DCDC_StepUp_SX1308-lm2596_module
- added Q? (x4): BC546, Package_TO_SOT_THT:TO-92_Inline, symbol Transistor_BJT:BC546
- added R? (x4): 4.7k, symbol Device:R
- added R? (x2): 1k, symbol Device:R
Connections:
- net +3V3: now also U2.3V3
- net +5V: now also R?.2, R?.2, R?.2, R?.2
- net CLK_LED: no longer J1.5 (Pin_5)
- net ENCODER1_A: now also U2.PB8; no longer U2.PB12
- net ENCODER1_B: now also U2.PB9; no longer U2.PB13
- net ENCODER2_A: now also U2.PB10; no longer U2.PB14
- net ENCODER2_B: now also U2.PB11; no longer U2.PB15
- net GND: now also Q?.3 (E), Q?.3 (E), Q?.3 (E), Q?.3 (E)
- net MOTOR1_EN: no longer U2.PA11
- net MOTOR1_INA: no longer U2.PA12
- net MOTOR1_INB: no longer U2.PA15
- net MOTOR1_PWM: now also U2.PB14; no longer U2.PB8
- net MOTOR2_EN: now also U2.PA11
- net MOTOR2_INA: now also U2.PA12
- net MOTOR2_INB: now also U2.PA15
- net MOTOR2_PWM: now also U2.PB15; no longer U2.PB9
- net SERVO1: now also R?.2; no longer M1.1 (PWM)
- net SERVO2: now also R?.2; no longer M2.1 (PWM)
- new net: M1.1 (PWM), Q?.1 (C), R?.1
- new net: M2.1 (PWM), Q?.1 (C), R?.1
- new net: Q?.2 (B), R?.1 (x2)
- new net: Q?.1 (C), Q?.2 (B), R?.1 (x2)
Other:
- moved on the sheet: C?, J1, J?, M1, M2, U1, U2

Commit message: PCB Layout inprog
Parts:
- removed J?: MPU6050, Connector_PinHeader_2.54mm:PinHeader_1x08_P2.54mm_Vertical, symbol Connector_Generic:Conn_01x08
- removed J?: Raspberry_Pi_2_3, Connector_PinHeader_2.54mm:PinHeader_2x20_P2.54mm_Vertical, symbol Connector:Raspberry_Pi_2_3
- removed J?: GPS, Connector_PinHeader_2.54mm:PinHeader_1x04_P2.54mm_Vertical, symbol Connector_Generic:Conn_01x04
- removed J?: BLUETOOTH, Connector_PinHeader_2.54mm:PinHeader_1x06_P2.54mm_Vertical, symbol Connector_Generic:Conn_01x06
- removed U2: ChinaBluePill, BLUEPILL:BluePill_STM32F103C, symbol D3_Board:ChinaBluePill-bluepill
- added J13: BUZZER_PIN, Connector_PinHeader_2.54mm:PinHeader_1x02_P2.54mm_Vertical, symbol Connector_Generic:Conn_01x02
- added J2: POWER_IN, TerminalBlock_Phoenix:TerminalBlock_Phoenix_PT-1,5-2-5.0-H_1x02_P5.00mm_Horizontal, symbol Connector_Generic:Conn_01x02
- added J4: Raspberry_connection, Connector_PinHeader_2.54mm:PinHeader_1x04_P2.54mm_Vertical, symbol Connector_Generic:Conn_01x04
- added J5: CURRENT_POWER_IN, TerminalBlock_Phoenix:TerminalBlock_Phoenix_PT-1,5-2-5.0-H_1x02_P5.00mm_Horizontal, symbol Connector_Generic:Conn_01x02
- added R1: 11k, Resistor_THT:R_Axial_DIN0207_L6.3mm_D2.5mm_P10.16mm_Horizontal, symbol Device:R
- added R2: 3.3k, Resistor_THT:R_Axial_DIN0207_L6.3mm_D2.5mm_P10.16mm_Horizontal, symbol Device:R
- added U1: ChinaBluePill-bluepill-D3_Board, BLUEPILL:BluePill_STM32F103C, symbol D3_Board:ChinaBluePill-bluepill-D3_Board
- added U3: GPS_NEO6M_module, D3_Board:GPS_NEO6M_module, symbol D3_Board:GPS_NEO6M_module
- added U4: MPU6050_module, D3_Board:MPU6050_module, symbol D3_Board:MPU6050_module
- C1: renamed from C?; value CP -> 1000uF; footprint (none) -> Capacitor_THT:CP_Radial_D10.0mm_P5.00mm
- J1: renamed from J?; footprint TerminalBlock:TerminalBlock_Altech_AK300-2_P5.00mm -> Connector_AMASS:AMASS_XT60-M_1x02_P7.20mm_Vertical
- J14, J15, J16, J17, J3: renamed from J?; footprint TerminalBlock:TerminalBlock_Altech_AK300-2_P5.00mm -> TerminalBlock_Phoenix:TerminalBlock_Phoenix_PT-1,5-2-5.0-H_1x02_P5.00mm_Horizontal
- J6: renamed from J1; footprint (none) -> Connector_PinHeader_2.54mm:PinHeader_1x05_P2.54mm_Vertical
- J8: renamed from J2; footprint Connector_PinHeader_2.54mm:PinHeader_1x06_P2.54mm_Vertical -> Connector_JST:JST_EH_B6B-EH-A_1x06_P2.50mm_Vertical
- J9: renamed from J3; footprint Connector_PinHeader_2.54mm:PinHeader_1x06_P2.54mm_Vertical -> Connector_JST:JST_EH_B6B-EH-A_1x06_P2.50mm_Vertical
- R10: renamed from R?; value 3.3K -> 3.3k; footprint (none) -> Resistor_THT:R_Axial_DIN0207_L6.3mm_D2.5mm_P10.16mm_Horizontal
- R3, R4, R5, R6, R7, R8: renamed from R?; footprint (none) -> Resistor_THT:R_Axial_DIN0207_L6.3mm_D2.5mm_P10.16mm_Horizontal
- R9: renamed from R?; value 1.7K -> 1.7k; footprint (none) -> Resistor_THT:R_Axial_DIN0207_L6.3mm_D2.5mm_P10.16mm_Horizontal
- U2: renamed from U1; footprint LM2596:lm2596_module -> D3_Board:LM2596_module; symbol D3_Board:YAAJ_DCDC_StepUp_SX1308-lm2596_module -> D3_Board:YAAJ_DCDC_StepUp_SX1308-lm2596_module-D3_Board
- gave numbers to parts that had none: 8
Connections:
- net +12V: now also J5.1 (Pin_1); no longer C1.1, J1.1 (Pin_1)
- net +3V3: now also U1.20 (3V3), U1.38 (3V3)
- net +5V: now also U1.18 (5V), U3.1 (VCC), U4.1 (VCC)
- net ACS: now also U1.5 (PA8)
- net CLK_LED: now also J6.5 (Pin_5), U1.30 (PA5)
- net CS_LED: now also U1.29 (PA4)
- net DOUT_LED: now also U1.32 (PA7)
- net ENCODER1_A: now also U1.16 (PB8)
- net ENCODER1_B: now also U1.17 (PB9)
- net ENCODER2_A: now also U1.35 (PB10)
- net ENCODER2_B: now also U1.36 (PB11)
- net GND: now also J1.1 (Pin_1), J13.2 (Pin_2), J2.2 (Pin_2), R2.2, U1.19 (GND), U1.39 (GND), U1.40 (GND), U3.4 (GND), U4.2 (GND); no longer J1.2 (Pin_2)
- net MOTOR1_CS: now also U1.25 (PA0)
- net MOTOR1_EN: now also U1.11 (PB3)
- net MOTOR1_INA: now also U1.12 (PB4)
- net MOTOR1_INB: now also U1.13 (PB5)
- net MOTOR1_PWM: now also U1.3 (PB14)
- net MOTOR2_CS: now also U1.26 (PA1)
- net MOTOR2_EN: now also U1.8 (PA11)
- net MOTOR2_INA: now also U1.9 (PA12)
- net MOTOR2_INB: now also U1.10 (PA15)
- net MOTOR2_PWM: now also U1.4 (PB15)
- net RX_GPS: now also J4.2 (Pin_2), U3.2 (RX)
- net RX_SERIAL: now also U1.6 (PA9)
- net SCL: now also J4.3 (Pin_3), U4.3 (SCL)
- net SDA: now also J4.4 (Pin_4), U4.4 (SDA)
- net SERVO1: now also U1.14 (PB6)
- net SERVO2: now also U1.15 (PB7)
- net TX_GPS: now also J4.1 (Pin_1), U3.3 (TX)
- net TX_SERIAL: now also U1.7 (PA10)
- new net: C1.1, J1.2 (Pin_2), J2.1 (Pin_1), J5.2 (Pin_2), R1.1
- new net AVS: R1.2, R2.1, U1.33 (PB0)
- new net BUZZER: J13.1 (Pin_1), U1.34 (PB1)
- no-connect marks 8 -> 16
Other:
- note added: "Bluepill será alimentado pelo\nconversor USB-TTL na raspberry\n"
- moved on the sheet: C1, J1, J10, J3, M1, M2, Q1, Q2, Q3, Q4, R10, R3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

Commit message: Finish traces
Connections:
- net ENCODER2_A: now also U1.36 (PB11); no longer U1.35 (PB10)
- net ENCODER2_B: now also U1.35 (PB10); no longer U1.36 (PB11)
Changed lines of the file:
@@
 ENCODER1_B
 Text Label 3000 6300 0    50   ~ 0
+ENCODER2_B
+Text Label 3000 6400 0    50   ~ 0
 ENCODER2_A
-Text Label 3000 6400 0    50   ~ 0
-ENCODER2_B
 Wire Wire Line
 	2900 6100 3000 6100

Commit message: Update main board Schematics
Other:
- note added: "<- Conexões da \nVNH2SP30 ->"
- note added: "Conector XT60 \npara bateria LiPo\n \n\n"
- note added: "Conector borne para\nalimentar com fonte\n \n\n"
- note added: "Ligar no sensor para\nleitura da corrente"
- note added: "Medição de tensão\nda bateria\n"
- note removed: "Bluepill será alimentado pelo\nconversor USB-TTL na raspberry\n"
- moved on the sheet: C1, J1, J10, J11, J12, J13, J14, J15, J16, J17, J2, J3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
